Commit message: Changed limits, edited code to work with Unity changes

File: chris_ur5_robotiq_config/config/gazebo_ur5_robotiq_3f_gripper.urdf (robot description, URDF)
Before this commit: robot ur5_robotiq_3f_gripper, 24 links, 23 joints
Joints:
- joint shoulder_lift_joint: limit lower=-3.141592653589793 upper=-0.0 effort=150.0 velocity=3.141592653589793 -> lower=-3.141592653589793 upper=0.0 effort=150.0 velocity=3.141592653589793
- joint wrist_1_joint: limit lower=-3.141592653589793 upper=0.0 effort=28.0 velocity=3.141592653589793 -> lower=-3.141592653589793 upper=3.141592653589793 effort=28.0 velocity=3.141592653589793
- joint wrist_2_joint: limit lower=0.0 upper=3.141592653589793 effort=28.0 velocity=3.141592653589793 -> lower=-3.141592653589793 upper=3.141592653589793 effort=28.0 velocity=3.141592653589793
